File: propeller-clock-smd.sch (KiCad schematic (older format))
At the start: 6 parts, among them IC1 ATMEGA328-P

Commit message: Added MAX7219 and LEDs
Connections:
- wire segments 56 -> 49
Changed lines of the file:
@@
 LIBS:74xgxx
 LIBS:74xx
+LIBS:c_integrated
+LIBS:propeller-clock-smd-cache
 EELAYER 25 0
 EELAYER END
@@
 $EndComp
 $Comp
-L VCC #PWR1
+L VCC #PWR101
 U 1 1 5474430A
 P 4450 2350
-F 0 "#PWR1" H 4450 2450 30  0001 C CNN
+F 0 "#PWR101" H 4450 2450 30  0001 C CNN
 F 1 "VCC" H 4450 2450 30  0000 C CNN
 F 2 "" H 4450 2350 60  0000 C CNN
@@
 $EndComp
 $Comp
-L GND #PWR2
+L GND #PWR102
 U 1 1 54744345
 P 4500 4950
-F 0 "#PWR2" H 4500 4950 30  0001 C CNN
+F 0 "#PWR102" H 4500 4950 30  0001 C CNN
 F 1 "GND" H 4500 4880 30  0001 C CNN
 F 2 "" H 4500 4950 60  0000 C CNN
@@
 $EndComp
 $Sheet
-S 6800 4450 550  500
+S 7250 5700 550  500
 U 547443D4
 F0 "LED" 50
 F1 "LED.sch" 50
-F2 "MOSI" I L 6800 4650 60
-F3 "SCK" I L 6800 4800 60
-F4 "LATCH" I L 6800 4500 60
+F2 "DIN" I L 7250 5900 60
+F3 "CLK" I L 7250 6050 60
+F4 "LOAD" I L 7250 5750 60
 $EndSheet
 $Sheet
@@
 $EndSheet
 $Comp
-L GND #PWR7
+L GND #PWR107
 U 1 1 54785E50
 P 8500 3800
-F 0 "#PWR7" H 8500 3800 30  0001 C CNN
+F 0 "#PWR107" H 8500 3800 30  0001 C CNN
 F 1 "GND" H 8500 3730 30  0001 C CNN
 F 2 "" H 8500 3800 60  0000 C CNN
@@
 $EndComp
 $Comp
-L VCC #PWR3
+L VCC #PWR103
 U 1 1 5478603D
 P 7850 1850
-F 0 "#PWR3" H 7850 1950 30  0001 C CNN
+F 0 "#PWR103" H 7850 1950 30  0001 C CNN
 F 1 "VCC" H 7850 1950 30  0000 C CNN
 F 2 "" H 7850 1850 60  0000 C CNN
@@
 $EndComp
 $Comp
-L GND #PWR4
+L GND #PWR104
 U 1 1 54786063
 P 7850 2500
-F 0 "#PWR4" H 7850 2500 30  0001 C CNN
+F 0 "#PWR104" H 7850 2500 30  0001 C CNN
 F 1 "GND" H 7850 2430 30  0001 C CNN
 F 2 "" H 7850 2500 60  0000 C CNN
@@
 	4600 4800 4500 4800
 Connection ~ 4500 4800
-Wire Wire Line
-	6500 4600 6650 4600
-Wire Wire Line
-	6650 4600 6650 4500
-Wire Wire Line
-	6650 4500 6800 4500
-Wire Wire Line
-	6500 4700 6700 4700
-Wire Wire Line
-	6700 4700 6700 4650
-Wire Wire Line
-	6700 4650 6800 4650
-Wire Wire Line
-	6500 4800 6800 4800
 Wire Wire Line
 	8500 3500 8500 3800
@@
 $EndComp
 $Comp
-L VCC #PWR6
+L VCC #PWR106
 U 1 1 547995F2
 P 8300 4000
-F 0 "#PWR6" H 8300 4100 30  0001 C CNN
+F 0 "#PWR106" H 8300 4100 30  0001 C CNN
 F 1 "VCC" H 8300 4100 30  0000 C CNN
 F 2 "" H 8300 4000 60  0000 C CNN
@@
 	8350 4450 8250 4450
 $Comp
-L GND #PWR5
+L GND #PWR105
 U 1 1 5479970A
 P 8250 5100
-F 0 "#PWR5" H 8250 5100 30  0001 C CNN
+F 0 "#PWR105" H 8250 5100 30  0001 C CNN
 F 1 "GND" H 8250 5030 30  0001 C CNN
 F 2 "" H 8250 5100 60  0000 C CNN
@@
 $EndComp
 $Comp
-L GND #PWR8
+L GND #PWR108
 U 1 1 54799730
 P 9750 5100
-F 0 "#PWR8" H 9750 5100 30  0001 C CNN
+F 0 "#PWR108" H 9750 5100 30  0001 C CNN
 F 1 "GND" H 9750 5030 30  0001 C CNN
 F 2 "" H 9750 5100 60  0000 C CNN
